File: Intro Project Alex Aarhus/Intro Project Alex Aarhus.kicad_sch (KiCad schematic)
At the start: 5 parts

Commit message: Finished Intro Project
Created and wired PCB board
Created Gerber files
Parts:
- removed R? (x2): R, symbol Device:R
- added BT1, BT2: 3V, Battery:BatteryHolder_LINX_BAT-HLD-012-SMT, symbol Device:Battery_Cell
- added D1: LED, LED_SMD:LED_0805_2012Metric, symbol Device:LED
- added R1: 5K, Resistor_SMD:R_0805_2012Metric, symbol Device:R_Small
- added R2: 10K, Resistor_SMD:R_0805_2012Metric, symbol Device:R_Small
- C1: renamed from C?; value C -> .01uF; footprint (none) -> Capacitor_SMD:C_0805_2012Metric
- C2: renamed from C?; value C -> 10uF; footprint (none) -> Capacitor_SMD:C_0805_2012Metric
- U1: renamed from U?; footprint Package_DIP:DIP-8_W7.62mm -> Package_SO:SOIC-8_3.9x4.9mm_P1.27mm
Connections:
- net GND: now also C2.1, BT2.2 (-), D1.1 (K); no longer C2.2
- net at U1.2 (TR), U1.6 (THR): now also C2.2, R2.2; no longer C2.1
- net at U1.7 (DIS): now also R1.2, R2.1
- net VCC: now reaches U1.4 (R), U1.8 (VCC)
- net VCC: now also BT1.1 (+), R1.1
- net at U1.3 (Q): now also D1.2 (A)
- new net: BT1.2 (-), BT2.1 (+)
Other:
- moved on the sheet: C1, C2
